File: dmx_led_strip_dimmer_32ch.sch (KiCad schematic (older format))
At the start: 104 parts, among them J1 Conn_01x11, J10 TEST_1P, J11 TEST_1P, J2 Conn_01x11, J3 Conn_01x10, J4 Conn_01x10, J5 Conn_01x03, J6 Conn_01x04, J8 TEST_1P, J9 TEST_1P, Q1 IRLZ44N, Q10 IRLZ44N, Q11 IRLZ44N, Q12 IRLZ44N, Q13 IRLZ44N, Q14 IRLZ44N, Q15 IRLZ44N, Q16 IRLZ44N, Q17 IRLZ44N, Q18 IRLZ44N, Q19 IRLZ44N, Q2 IRLZ44N, Q20 IRLZ44N, Q21 IRLZ44N, Q22 IRLZ44N, Q23 IRLZ44N, Q24 IRLZ44N, Q25 IRLZ44N, Q26 IRLZ44N, Q27 IRLZ44N, Q28 IRLZ44N, Q29 IRLZ44N, Q3 IRLZ44N, Q30 IRLZ44N, Q31 IRLZ44N, Q32 IRLZ44N, Q4 IRLZ44N, Q5 IRLZ44N, Q6 IRLZ44N, Q7 IRLZ44N, Q8 IRLZ44N, Q9 IRLZ44N, U1 74HC04, U10 SN75176, U11 L7805, U2 74HC04, U3 74HC04, U4 74HC04, U5 74HC04, U6 74HC04, U7 TLC5940PWP, U8 TLC5940PWP, U9 ArduinoMini

Commit message: Updated schematic to KiCad 5
Parts:
- removed J1, J2: Conn_01x11, Connectors_Terminal_Blocks:TerminalBlock_Pheonix_MKDS1.5-11pol, symbol Conn_01x11
- removed J10, J11, J8, J9: TEST_1P, Mounting_Holes:MountingHole_3.2mm_M3_ISO7380_Pad, symbol TEST_1P
- removed J3, J4: Conn_01x10, Connectors_Terminal_Blocks:TerminalBlock_Pheonix_MKDS1.5-10pol, symbol Conn_01x10
- removed J5: Conn_01x03, Connectors_Terminal_Blocks:TerminalBlock_Pheonix_MKDS1.5-3pol, symbol Conn_01x03
- removed J6: Conn_01x04, Connectors_Terminal_Blocks:TerminalBlock_Pheonix_MKDS1.5-4pol, symbol Conn_01x04
- removed Q1, Q10, Q11, Q12, Q13, Q14, Q15, Q16, Q17, Q18, Q19, Q2, Q20, Q21, Q22, Q23, Q24, Q25, Q26, Q27, Q28, Q29, Q3, Q30, Q31, Q32, Q4, Q5, Q6, Q7, Q8, Q9: IRLZ44N, TO_SOT_Packages_THT:TO-220_Vertical, symbol IRLZ44N
- removed U10: SN75176, Housings_SOIC:SOIC-8_3.9x4.9mm_Pitch1.27mm, symbol SN75176
- removed U11: L7805, TO_SOT_Packages_THT:TO-220-3_Vertical, symbol L7805
- removed U7, U8: TLC5940PWP, Housings_SSOP:TSSOP-28_4.4x9.7mm_Pitch0.65mm, symbol TLC5940PWP
- removed U9: ArduinoMini, Housings_DIP:DIP-24_W15.24mm_LongPads, symbol ArduinoMini
- added J1: OUT1, TerminalBlock_Phoenix:TerminalBlock_Phoenix_MKDS-1,5-11_1x11_P5.00mm_Horizontal, symbol Connector_Generic:Conn_01x11
- added J10, J11, J8, J9: TEST_1P, MountingHole:MountingHole_3.2mm_M3_ISO7380_Pad, symbol Connector:TestPoint
- added J2: OUT2, TerminalBlock_Phoenix:TerminalBlock_Phoenix_MKDS-1,5-11_1x11_P5.00mm_Horizontal, symbol Connector_Generic:Conn_01x11
- added J3: OUT3, TerminalBlock_Phoenix:TerminalBlock_Phoenix_MKDS-1,5-10_1x10_P5.00mm_Horizontal, symbol Connector_Generic:Conn_01x10
- added J4: OUT4, TerminalBlock_Phoenix:TerminalBlock_Phoenix_MKDS-1,5-10_1x10_P5.00mm_Horizontal, symbol Connector_Generic:Conn_01x10
- added J5: DMX, TerminalBlock_Phoenix:TerminalBlock_Phoenix_MKDS-1,5-3_1x03_P5.00mm_Horizontal, symbol Connector_Generic:Conn_01x03
- added J6: PWR, TerminalBlock_Phoenix:TerminalBlock_Phoenix_MKDS-1,5-4_1x04_P5.00mm_Horizontal, symbol Connector_Generic:Conn_01x04
- added Q1, Q10, Q11, Q12, Q13, Q14, Q15, Q16, Q17, Q18, Q19, Q2, Q20, Q21, Q22, Q23, Q24, Q25, Q26, Q27, Q28, Q29, Q3, Q30, Q31, Q32, Q4, Q5, Q6, Q7, Q8, Q9: IRLZ44N, Package_TO_SOT_THT:TO-220-3_Vertical, symbol Transistor_FET:IRLZ44N
- added U10: SN75LBC176P, Package_DIP:DIP-8_W7.62mm, symbol Interface_UART:SN75LBC176P
- added U11: L7805, Package_TO_SOT_THT:TO-220-3_Vertical, symbol Regulator_Linear:L7805
- added U7, U8: TLC5940PWP, Package_SO:HTSSOP-28-1EP_4.4x9.7mm_P0.65mm_EP3.4x9.5mm_Mask2.4x6.17mm_ThermalVias, symbol Driver_LED:TLC5940PWP
- added U9: ArduinoMini, Package_DIP:DIP-24_W15.24mm_LongPads, symbol arduinomini:ArduinoMini
- C1, C10, C11, C15, C16, C2, C3, C4, C5, C6, C7, C8, C9: symbol C -> Device:C
- D1, D2: symbol D_Zener -> Device:D_Zener
- JP1: symbol Jumper_NO_Small -> Device:Jumper_NO_Small
- R1, R10, R11, R12, R13, R14, R15, R16, R17, R18, R19, R2, R20, R21, R22, R23, R24, R25, R26, R27, R28, R29, R3, R30, R31, R32, R33, R34, R35, R4, R5, R6, R7, R8, R9: symbol R -> Device:R
- U1, U2, U3, U4, U5, U6: symbol 74HC04 -> 74xx:74HC04
Connections:
- wire segments 417 -> 493
Other:
- moved on the sheet: D1, D2, JP1, R35

Commit message: Archived project for better portability
Parts:
- C1, C10, C11, C15, C16, C2, C3, C4, C5, C6, C7, C8, C9: symbol Device:C -> archive:Device_C
- D1, D2: symbol Device:D_Zener -> archive:Device_D_Zener
- J1, J2: symbol Connector_Generic:Conn_01x11 -> archive:Connector_Generic_Conn_01x11
- J10, J11, J8, J9: symbol Connector:TestPoint -> archive:Connector_TestPoint
- J3, J4: symbol Connector_Generic:Conn_01x10 -> archive:Connector_Generic_Conn_01x10
- J5: symbol Connector_Generic:Conn_01x03 -> archive:Connector_Generic_Conn_01x03
- J6: symbol Connector_Generic:Conn_01x04 -> archive:Connector_Generic_Conn_01x04
- JP1: symbol Device:Jumper_NO_Small -> archive:Device_Jumper_NO_Small
- Q1, Q10, Q11, Q12, Q13, Q14, Q15, Q16, Q17, Q18, Q19, Q2, Q20, Q21, Q22, Q23, Q24, Q25, Q26, Q27, Q28, Q29, Q3, Q30, Q31, Q32, Q4, Q5, Q6, Q7, Q8, Q9: symbol Transistor_FET:IRLZ44N -> archive:Transistor_FET_IRLZ44N
- R1, R10, R11, R12, R13, R14, R15, R16, R17, R18, R19, R2, R20, R21, R22, R23, R24, R25, R26, R27, R28, R29, R3, R30, R31, R32, R33, R34, R35, R4, R5, R6, R7, R8, R9: symbol Device:R -> archive:Device_R
- U1, U2, U3, U4, U5, U6: symbol 74xx:74HC04 -> archive:74xx_74HC04
- U10: symbol Interface_UART:SN75LBC176P -> archive:Interface_UART_SN75LBC176P
- U11: symbol Regulator_Linear:L7805 -> archive:Regulator_Linear_L7805
- U7, U8: symbol Driver_LED:TLC5940PWP -> archive:Driver_LED_TLC5940PWP
- U9: symbol arduinomini:ArduinoMini -> archive:arduinomini_ArduinoMini
